File: n2adr.sch (KiCad schematic (older format))
At the start: 106 parts, among them CN1 STEREO, CN2 Conn_01x20, CN3 SMA, CN4 SMA, CN5 SMA, CN6 SMA, CN7 SMA, CN8 SMA, J1 coax rf low, J2 coax rx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

Commit message: upgrade to Kicad 5.x, 2 layers less
Connections:
- net GND: now also RV1.3
Changed lines of the file:
@@
 Connection ~ 6550 6300
 Wire Wire Line
-	5100 6300 5650 6300
+	5100 6300 5250 6300
 Connection ~ 5650 5600
 Wire Wire Line
@@
 Wire Wire Line
 	5450 4700 5750 4700
+Wire Wire Line
+	5250 6250 5250 6300
+Connection ~ 5250 6300
+Wire Wire Line
+	5250 6300 5650 6300
 $EndSCHEMATC
